Commit message: Working circle

File: urdf/my_robot.urdf (robot description, URDF)
Before this commit: robot my_robot, 3 links, 2 joints
Links:
- link link1: geometry 
- link link2: geometry visual cylinder length=1 radius=.05
- link link3: geometry visual cylinder length=1 radius=.05
Joints:
- joint joint1: origin xyz=1 0 0 rpy=0 0 0 -> xyz=0 0 0 rpy=0 0 0

Commit message: working params, working markers

File: urdf/my_robot.urdf (robot description, URDF)
Before this commit: robot my_robot, 3 links, 2 joints
Links:
- added link link4
Joints:
- added joint joint3: type continuous, parent link3, child link4, origin xyz=1 0 0 rpy=0 0 0, axis 0 0 1
